Commit message: dh corregido. control cinematico de posicion completo. control cinematico de orientacion incompleto (no es necesario). instalacion de rbdl e implementacion de codigo de control dinamico (falta corregir).

File: robot_description/urdf/robot_description.urdf (robot description, URDF)
Before this commit: robot edo, 8 links, 7 joints
Links:
- link cylinder_link: geometry collision cylinder length=0.25 radius=0.033; visual cylinder length=0.25 radius=0.033
Joints:
- joint joint_1: limit (none) -> lower=-3.12 upper=3.12 effort=2.75 velocity=0.4; type continuous -> revolute
- joint joint_2: limit (none) -> lower=-1.73 upper=1.73 effort=2.75 velocity=0.4; type continuous -> revolute
- joint joint_3: limit (none) -> lower=-1.73 upper=1.73 effort=2.75 velocity=0.4; type continuous -> revolute
- joint joint_4: limit (none) -> lower=-3.12 upper=3.12 effort=2.75 velocity=0.59; origin xyz=0.0088 -0.1588 0 rpy=-1.5708 0 0 -> xyz=0 -0.121 0 rpy=-1.5708 0 0; type continuous -> revolute
- joint joint_5: limit (none) -> lower=-1.81 upper=1.81 effort=2.75 velocity=0.59; type continuous -> revolute
- joint joint_6: limit (none) -> lower=-3.12 upper=3.12 effort=2.75 velocity=0.59; type continuous -> revolute
- joint prismatic_joint: limit lower=0.0 upper=0.5 effort=50 velocity=1.0 -> lower=0.0 upper=0.1 effort=5 velocity=0.5; origin xyz=0 0 0.0 rpy=0 0 0 -> xyz=0.0 -0.2 0 rpy=0 0 0

Commit message: control dinamico completo. se podria mejorar rendimiento. falta implementar un modelo de control mas y validacion en gazebo.

File: robot_description/urdf/robot_description.urdf (robot description, URDF)
Before this commit: robot edo, 8 links, 7 joints
Links:
- link cylinder_link: mass 1.0 -> 0.01
Joints:
- joint prismatic_joint: limit lower=0.0 upper=0.1 effort=5 velocity=0.5 -> lower=0.0 upper=0.1 effort=2.75 velocity=0.5

Commit message: gazebo listo para validacion. falta implementar control dinamico en gazebo. se centralizaron los controladores del yaml.

File: robot_description/urdf/robot_description.urdf (robot description, URDF)
Before this commit: robot edo, 8 links, 7 joints
Links:
- added link world
Joints:
- added joint base_to_world: type fixed, parent world, child base_link, origin xyz=0 0 0 rpy=0 0 0
